File: DormLock.kicad_pcb (KiCad board)
At the start: 2 copper layers, 68.9 x 82.5 mm, 48 parts, among them J1 Conn_02x03_Odd_Even, J2 Conn_01x05, J4 Conn_01x03, J5 Conn_01x02, J6 Conn_01x15, J7 Conn_01x15, J8 Conn_01x08, J9 USB_C_Receptacle, Q1 Q_NPN_EBC, Q2 Q_PMOS_GSD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

Commit message: V0.2
Parts:
- added R13: 100k, Resistor_SMD:R_0603_1608Metric, F.Cu at (168.0, 92.9)
- added R14: 5.1k, Resistor_SMD:R_0603_1608Metric, B.Cu at (194.4, 114.7)
- added R15: 5.1k, Resistor_SMD:R_0603_1608Metric, B.Cu at (193.8, 111.1)
- C15, C9: value 1000uf -> 470uf
- C6: value 1nf -> 1uf
- C7: value 2.2nf -> 2.2uf
- Q2: footprint Package_TO_SOT_SMD:SOT-23 -> KisonCommon:DFN-8-1EP_3x3mm_P0.65mm_EP1.7x2.05mm
- R10: value 470 -> 2.2k
- moved Q2 3.83 mm to (173.5, 87.7)
Connections:
- J9 pad B6: Net-(J9-PadB6) -> Net-(J9-PadA6)
- J9 pad B7: Net-(J9-PadB7) -> Net-(J9-PadA7)
Routing:
- net Net-(J9-PadA7): track 0.00 -> 3.67 mm
- net Net-(J9-PadA6): track 0.00 -> 3.43 mm
- net /VOutput: track 49.0 -> 52.3 mm
- net Net-(J9-PadA5): track 0.00 -> 3.11 mm, vias 0 -> 1
- net Net-(Q1-Pad2): track 44.1 -> 46.8 mm
- net Net-(J9-PadB5): track 0.00 -> 2.26 mm, vias 0 -> 1
Other:
- board text added: "KisonHe"

Commit message: V0.25
Parts:
- moved C6 4.11 mm to (149.7, 64.5), turned to 180 degrees
- moved C7 2.04 mm to (167.0, 68.6), turned to 0 degrees
- moved C3 1.88 mm to (158.6, 97.4)
- moved R15 1.77 mm to (195.6, 111.0)
- moved R14 1.61 mm to (196.0, 114.7)
Routing:
- net +5V: track 102.9 -> 119.7 mm, vias 3 -> 2
- net +3V3: track 229.7 -> 243.0 mm, vias 8 -> 7
- net GND: track 3.80 -> 14.5 mm
- net Net-(R8-Pad1): track 2.33 -> 4.76 mm
- net Net-(Q3-Pad2): track 5.47 -> 7.74 mm
- net /STM_NRST: track 93.6 -> 95.4 mm
- net Net-(J9-PadB5): track 2.26 -> 4.02 mm
- net Net-(J9-PadA5): track 3.11 -> 4.71 mm
- net Vdrive: track 33.9 -> 32.5 mm, vias 2 -> 1
- net +BATT: track 31.2 -> 30.3 mm
- net /VOutput: track 52.3 -> 53.1 mm
- net /UART_32RX: track 28.0 -> 28.6 mm

Commit message: V0.29
Parts:
- L1: footprint Inductor_SMD:L_1008_2520Metric -> Inductor_SMD:L_6.3x6.3_H3; moved to B.Cu
- moved L1 0.58 mm to (173.7, 67.0)
Routing:
- net +5V: track 119.7 -> 126.1 mm
- net Net-(C14-Pad1): track 10.1 -> 14.9 mm
Changed lines of the file:
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@@
     (thickness 1.6)
     (drawings 11)
-    (tracks 335)
+    (tracks 341)
     (zones 0)
     (modules 51)
@@
   )
   (setup
-    (last_trace_width 0.2)
+    (last_trace_width 0.8)
     (user_trace_width 0.2)
     (user_trace_width 0.5)
+    (user_trace_width 0.8)
     (user_trace_width 1)
     (user_trace_width 1.5)
@@
     (add_net Vdrive)
   )
+  (module Inductor_SMD:L_6.3x6.3_H3 (layer B.Cu)
+    (at 173.67 66.99 270)
+    (descr "Choke, SMD, 6.3x6.3mm 3mm height")
+    (tags "Choke SMD")
+    (attr smd)
+    (fp_text reference L1 (at 0 4.45 270) (layer B.SilkS)
+      (effects (font (size 1 1) (thickness 0.15)) (justify mirror))
+    )
+    (fp_text value 4.7uh (at 0 -4.45 270) (layer B.Fab)
+      (effects (font (size 1 1) (thickness 0.15)) (justify mirror))
+    )
+    (fp_arc (start 0 0) (end 1.91 -1.91) (angle -90) (layer B.Fab) (width 0.1))
+    (fp_arc (start 0 0) (end -1.91 1.91) (angle -90) (layer B.Fab) (width 0.1))
+    (fp_text user %R (at 0 0 270) (layer B.Fab)
+      (effects (font (size 1 1) (thickness 0.15)) (justify mirror))
+    )
+    (fp_line (start 3.3 -1.5) (end 3.3 -3.2) (layer B.SilkS) (width 0.12))
+    (fp_line (start 3.3 -3.2) (end -3.3 -3.2) (layer B.SilkS) (width 0.12))
+    (fp_line (start -3.3 -3.2) (end -3.3 -1.5) (layer B.SilkS) (width 0.12))
+    (fp_line (start -3.3 1.5) (end -3.3 3.2) (layer B.SilkS) (width 0.12))
+    (fp_line (start -3.3 3.2) (end 3.3 3.2) (layer B.SilkS) (width 0.12))
+    (fp_line (start 3.3 3.2) (end 3.3 1.5) (layer B.SilkS) (width 0.12))
+    (fp_line (start -3.75 3.4) (end -3.75 -3.4) (layer B.CrtYd) (width 0.05))
+    (fp_line (start -3.75 -3.4) (end 3.75 -3.4) (layer B.CrtYd) (width 0.05))
+    (fp_line (start 3.75 -3.4) (end 3.75 3.4) (layer B.CrtYd) (width 0.05))
+    (fp_line (start 3.75 3.4) (end -3.75 3.4) (layer B.CrtYd) (width 0.05))
+    (fp_line (start 3.15 -3.15) (end 3.15 -1.5) (layer B.Fab) (width 0.1))
+    (fp_line (start 3.15 3.15) (end 3.15 1.5) (layer B.Fab) (width 0.1))
+    (fp_line (start -3.15 -3.15) (end -3.15 -1.5) (layer B.Fab) (width 0.1))
+    (fp_line (start -3.15 3.15) (end -3.15 1.5) (layer B.Fab) (width 0.1))
+    (fp_line (start -3.15 3.15) (end 3.15 3.15) (layer B.Fab) (width 0.1))
+    (fp_line (start -3.15 -3.15) (end 3.15 -3.15) (layer B.Fab) (width 0.1))
+    (pad 2 smd rect (at 2.75 0 270) (size 1.5 2.4) (layers B.Cu B.Paste B.Mask)
+      (net 25 "Net-(C14-Pad1)"))
+    (pad 1 smd rect (at -2.75 0 270) (size 1.5 2.4) (layers B.Cu B.Paste B.Mask)
+      (net 6 +5V))
+    (model ${KISYS3DMOD}/Inductor_SMD.3dshapes/L_6.3x6.3_H3.wrl
+      (at (xyz 0 0 0))
+      (scale (xyz 1 1 1))
+      (rotate (xyz 0 0 0))
+    )
+  )
   (module Resistor_SMD:R_0603_1608Metric (layer B.Cu)
     (at 195.55 111.01 180)
@@
     (pad MP smd rect (at 3.65 1.4 180) (size 1.8 2.2) (layers F.Cu F.Paste F.Mask))
     (model ${KISYS3DMOD}/Connector_FFC-FPC.3dshapes/Hirose_FH12-8S-0.5SH_1x08-1MP_P0.50mm_Horizontal.wrl
-      (at (xyz 0 0 0))
-      (scale (xyz 1 1 1))
-      (rotate (xyz 0 0 0))
-    )
-  )
-  (module Inductor_SMD:L_1008_2520Metric (layer F.Cu)
-    (at 174.244 67.056 270)
-    (descr "Inductor SMD 1008 (2520 Metric), square (rectangular) end terminal, IPC_7351 nominal, (Body size source: https://ecsxtal.com/store/pdf/ECS-MPI2520-SMD-POWER-INDUCTOR.pdf), generated with kicad-footprint-generator")
-    (tags inductor)
-    (attr smd)
-    (fp_text reference L1 (at 0 -2.05 90) (layer F.SilkS)
-      (effects (font (size 1 1) (thickness 0.15)))
-    )
-    (fp_text value 4.7uh (at 0 2.05 90) (layer F.Fab)
-      (effects (font (size 1 1) (thickness 0.15)))
-    )
-    (fp_line (start 1.95 1.35) (end -1.95 1.35) (layer F.CrtYd) (width 0.05))
-    (fp_line (start 1.95 -1.35) (end 1.95 1.35) (layer F.CrtYd) (width 0.05))
-    (fp_line (start -1.95 -1.35) (end 1.95 -1.35) (layer F.CrtYd) (width 0.05))
-    (fp_line (start -1.95 1.35) (end -1.95 -1.35) (layer F.CrtYd) (width 0.05))
-    (fp_line (start -0.261252 1.11) (end 0.261252 1.11) (layer F.SilkS) (width 0.12))
-    (fp_line (start -0.261252 -1.11) (end 0.261252 -1.11) (layer F.SilkS) (width 0.12))
-    (fp_line (start 1.25 1) (end -1.25 1) (layer F.Fab) (width 0.1))
-    (fp_line (start 1.25 -1) (end 1.25 1) (layer F.Fab) (width 0.1))
-    (fp_line (start -1.25 -1) (end 1.25 -1) (layer F.Fab) (width 0.1))
-    (fp_line (start -1.25 1) (end -1.25 -1) (layer F.Fab) (width 0.1))
-    (fp_text user %R (at 0 0 90) (layer F.Fab)
-      (effects (font (size 0.62 0.62) (thickness 0.09)))
-    )
-    (pad 2 smd roundrect (at 1.075 0 270) (size 1.25 2.2) (layers F.Cu F.Paste F.Mask) (roundrect_rratio 0.2)
-      (net 25 "Net-(C14-Pad1)"))
-    (pad 1 smd roundrect (at -1.075 0 270) (size 1.25 2.2) (layers F.Cu F.Paste F.Mask) (roundrect_rratio 0.2)
-      (net 6 +5V))
-    (model ${KISYS3DMOD}/Inductor_SMD.3dshapes/L_1008_2520Metric.wrl
       (at (xyz 0 0 0))
       (scale (xyz 1 1 1))
@@
   (segment (start 187.77 112.27) (end 189.69 110.35) (width 0.5) (layer F.Cu) (net 6))
   (segment (start 187.77 115.25) (end 187.77 112.27) (width 0.5) (layer F.Cu) (net 6))
+  (segment (start 167.4 64.24) (end 167.35 64.29) (width 1) (layer B.Cu) (net 6))
+  (segment (start 173.67 64.24) (end 167.4 64.24) (width 1) (layer B.Cu) (net 6))
   (segment (start 159.90001 95.444311) (end 152.085699 87.63) (width 0.2) (layer F.Cu) (net 7))
   (segment (start 159.90001 99.611691) (end 159.90001 95.444311) (width 0.2) (layer F.Cu) (net 7))
@@
   (segment (start 180.253 66.7595) (end 181.2125 65.8) (width 0.25) (layer F.Cu) (net 24))
   (segment (start 180.253 67.376) (end 180.253 66.7595) (width 0.25) (layer F.Cu) (net 24))
-  (via (at 174.244 68.326) (size 0.8) (drill 0.4) (layers F.Cu B.Cu) (net 25))
+  (via (at 173.63 67.29) (size 0.8) (drill 0.4) (layers F.Cu B.Cu) (net 25))
   (segment (start 180.253 68.326) (end 180.253 68.326) (width 0.2) (layer F.Cu) (net 25))
-  (via (at 180.253 68.326) (size 0.8) (drill 0.4) (layers F.Cu B.Cu) (net 25))
-  (segment (start 174.244 68.326) (end 180.253 68.326) (width 0.2) (layer B.Cu) (net 25))
-  (segment (start 181.113 68.326) (end 180.253 68.326) (width 0.25) (layer F.Cu) (net 25))
-  (segment (start 182.7875 66.6515) (end 181.113 68.326) (width 0.25) (layer F.Cu) (net 25))
-  (segment (start 182.7875 65.8) (end 182.7875 66.6515) (width 0.25) (layer F.Cu) (net 25))
+  (via (at 181.78 67.68) (size 0.8) (drill 0.4) (layers F.Cu B.Cu) (net 25))
+  (segment (start 173.63 69.7) (end 173.67 69.74) (width 1) (layer B.Cu) (net 25))
+  (segment (start 173.63 67.29) (end 173.63 69.7) (width 1) (layer B.Cu) (net 25))
+  (segment (start 181.134 68.326) (end 181.78 67.68) (width 0.8) (layer F.Cu) (net 25))
+  (segment (start 180.253 68.326) (end 181.134 68.326) (width 0.8) (layer F.Cu) (net 25))
+  (segment (start 182.7875 66.6725) (end 182.7875 65.8) (width 0.8) (layer F.Cu) (net 25))
+  (segment (start 181.78 67.68) (end 182.7875 66.6725) (width 0.8) (layer F.Cu) (net 25))
+  (segment (start 181.39 67.29) (end 181.78 67.68) (width 0.8) (layer B.Cu) (net 25))
+  (segment (start 173.63 67.29) (end 181.39 67.29) (width 0.8) (layer B.Cu) (net 25))
   (segment (start 177.107998 68.326) (end 177.633 68.326) (width 0.2) (layer F.Cu) (net 64))
   (segment (start 175.514 69.919998) (end 177.107998 68.326) (width 0.2) (layer F.Cu) (net 64))

Commit message: V1.0
Parts:
- J2: footprint Connector_PinHeader_1.27mm:PinHeader_1x05_P1.27mm_Vertical -> Connector_PinHeader_2.54mm:PinHeader_1x05_P2.54mm_Vertical
- Q3: value Q_NPN_EBC -> Q_PMOS_GSD; footprint Package_TO_SOT_SMD:SOT-23 -> KisonCommon:DFN-8-1EP_3x3mm_P0.65mm_EP1.7x2.05mm
- moved Q3 6.41 mm to (154.7, 120.1)
- moved J2 0.16 mm to (167.7, 126.4)
Connections:
- Q3 pad 1: /LEDA -> Net-(Q3-Pad1)
- Q3 pad 2: Net-(Q3-Pad2) -> +3V3
- Q3 pad 3: +3V3 -> /LEDA
- R11 pad 1: Net-(Q3-Pad2) -> Net-(Q3-Pad1)
- R12 pad 1: Net-(Q3-Pad2) -> Net-(Q3-Pad1)
Routing:
- net /STM_NRST: track 95.4 -> 113.9 mm
- net Net-(Q3-Pad1): track 0.00 -> 11.5 mm, vias 0 -> 2
- net Net-(Q3-Pad2): track 7.74 -> 0.00 mm, vias 2 -> 0
- net /LEDA: track 22.2 -> 17.7 mm
- net /STM_SWCLK: track 44.1 -> 47.3 mm
- net /STM_SWDIO: track 45.9 -> 47.6 mm
- net +3V3: track 243.0 -> 244.5 mm

Commit message: V1.1
Parts:
- C14, C6, C7, R2, R5, R6, U1, U2: moved to B.Cu
- L1: moved to F.Cu
- moved C6 56.5 mm to (188.5, 105.6), turned to 0 degrees
- moved C13 51.2 mm to (177.1, 110.2), turned to 0 degrees
- moved H2 46.9 mm to (137.9, 76.5)
- moved C12 46.7 mm to (177.1, 107.5), turned to 0 degrees
- moved U1 46.2 mm to (180.5, 108.8)
- moved C7 44.0 mm to (173.9, 112.1), turned to 180 degrees
- moved C11 42.5 mm to (177.1, 104.8), turned to 0 degrees
- moved R3 40.4 mm to (173.7, 102.7), turned to 270 degrees
- moved C15 38.7 mm to (175.1, 79.8), turned to 90 degrees
- moved R4 36.8 mm to (177.1, 101.9), turned to 0 degrees
- moved C14 36.3 mm to (178.7, 101.9)
- moved SW1 35.1 mm to (172.4, 137.2)
- moved L1 31.5 mm to (182.9, 97.1), turned to 90 degrees
- moved C16 31.3 mm to (193.2, 79.4), turned to 90 degrees
- moved R6 29.6 mm to (169.6, 100.5), turned to 270 degrees
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Connections:
- U3 pad 34: /STM_SWCLK -> /STM_SWDIO
- U3 pad 37: /STM_SWDIO -> /STM_SWCLK
Routing:
- net +5V: track 126.1 -> 58.3 mm
- net +3V3: track 244.5 -> 177.3 mm
- net /STM_NRST: track 113.9 -> 85.5 mm
- net /VOutput: track 53.1 -> 38.2 mm
- net /STM_SWCLK: track 47.3 -> 59.1 mm, vias 0 -> 1
- net Vdrive: track 32.5 -> 37.6 mm, vias 1 -> 2
- net Net-(C14-Pad2): track 1.97 -> 4.36 mm
- net /STM_SWDIO: track 47.6 -> 45.2 mm
- net +BATT: track 30.3 -> 32.3 mm, vias 0 -> 1
- net Net-(R5-Pad1): track 7.97 -> 6.65 mm
- net Net-(C11-Pad1): track 8.30 -> 9.38 mm, vias 0 -> 1
- net Net-(C14-Pad1): track 14.9 -> 14.2 mm, vias 2 -> 1
Other:
- board size 68.9 x 82.5 mm -> 68.8 x 67.6 mm

Commit message: V1.2
Parts:
- added H13: 1mm Hole, KisonCommon:1mm Hole, F.Cu at (117.8, 81.7)
- added H13: 1mm Hole, KisonCommon:1mm Hole, F.Cu at (117.8, 83.0)
- added H13: 1mm Hole, KisonCommon:1mm Hole, F.Cu at (117.8, 84.2)
- added H13: 1mm Hole, KisonCommon:1mm Hole, F.Cu at (116.5, 81.7)
- added H13: 1mm Hole, KisonCommon:1mm Hole, F.Cu at (116.5, 83.0)
- added H13: 1mm Hole, KisonCommon:1mm Hole, F.Cu at (116.5, 84.2)
- added H5: MountingHole, MountingHole:MountingHole_2.2mm_M2_DIN965, F.Cu at (123.3, 87.1)
- added H6: MountingHole, MountingHole:MountingHole_2.2mm_M2_DIN965, F.Cu at (152.7, 67.5)
- added H7: MountingHole, MountingHole:MountingHole_2.2mm_M2_DIN965, F.Cu at (123.3, 78.8)
- added J10: Conn_02x03_Odd_Even, Connector_PinHeader_1.27mm:PinHeader_2x03_P1.27mm_Vertical, F.Cu at (147.2, 62.0)
- added R16: 10k, Resistor_SMD:R_0603_1608Metric, B.Cu at (146.8, 107.8)
- added R17: 10k, Resistor_SMD:R_0603_1608Metric, B.Cu at (149.2, 115.0)
- added R18: 5.1k, Resistor_SMD:R_0603_1608Metric, B.Cu at (145.8, 115.0)
- added R19: 10k, Resistor_SMD:R_0603_1608Metric, B.Cu at (150.7, 109.3)
- added U4: LM321, Package_TO_SOT_SMD:SOT-23-5, B.Cu at (147.2, 111.2)
- H1, H2, H3, H4: footprint MountingHole:MountingHole_3mm -> MountingHole:MountingHole_2.2mm_M2_DIN965
- J8, R13: moved to B.Cu
- Q1: value Q_NPN_EBC -> Q_NPN_BEC
- moved H1 46.1 mm to (174.8, 118.8)
- moved R13 14.0 mm to (163.8, 79.5), turned to 180 degrees
- moved H2 11.0 mm to (144.3, 67.5), turned to 90 degrees
- moved J1 4.95 mm to (160.6, 136.2)
- moved J8 1.64 mm to (151.5, 129.9)
- moved Q1 0.11 mm to (168.9, 88.6)
Connections:
- J4 pad 1: /VOutput -> /STEER_PWM
- J4 pad 2: /STEER_PWM -> /VOutput
- J5 pad 1: +BATT -> GND
- J5 pad 2: GND -> +BATT
- Q1 pad 1: GND -> Net-(Q1-Pad1)
- Q1 pad 2: Net-(Q1-Pad2) -> GND
- R13 pad 1: Net-(Q1-Pad2) -> Net-(Q1-Pad1)
- R9 pad 1: Net-(Q1-Pad2) -> Net-(Q1-Pad1)
- U3 pad 12: Net-(U3-Pad12) -> /RESET
Routing:
- net +3V3: track 177.3 -> 273.7 mm, vias 7 -> 8
- net +BATT: track 32.3 -> 97.8 mm, vias 1 -> 2
- net Net-(Q1-Pad2): track 46.8 -> 0.00 mm
- net Net-(Q1-Pad1): track 0.00 -> 44.6 mm, vias 0 -> 1
- net /RESET: track 0.00 -> 32.4 mm, vias 0 -> 1
- net /BATT_AD: track 0.00 -> 15.0 mm, vias 0 -> 1
- net Net-(R16-Pad1): track 0.00 -> 12.6 mm
- net /LEDA: track 17.7 -> 12.4 mm, vias 0 -> 1
- net /DC: track 27.7 -> 22.6 mm, vias 0 -> 1
- net Net-(R17-Pad2): track 0.00 -> 4.73 mm
- net /SDA: track 27.7 -> 23.3 mm, vias 0 -> 1
- net /SCL: track 27.8 -> 23.8 mm, vias 0 -> 1
- net /STM_SWDIO: track 45.2 -> 48.9 mm
- net GND: track 14.5 -> 17.4 mm
- net /CS: track 27.7 -> 25.4 mm, vias 0 -> 1
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Other:
- board size 68.8 x 67.6 mm -> 84.9 x 81.7 mm

Commit message: Update UART IRQ
Connections:
- J6 pad 3: /UART_32TX -> /UART_32RX
- J6 pad 4: /UART_32RX -> /UART_32TX
Routing:
- net /UART_32RX: track 28.6 -> 31.4 mm
- net /UART_32TX: track 30.9 -> 28.2 mm

Commit message: V2.0
Routing:
- net Vdrive: track 37.6 -> 34.1 mm
