File: DormLock.sch (KiCad schematic (older format))
At the start: 48 parts, among them J1 Conn_02x03_Odd_Even, J2 Conn_01x05, J4 Conn_01x03, J5 Conn_01x02, J6 Conn_01x15, J7 Conn_01x15, J8 Conn_01x08, J9 USB_C_Receptacle, Q1 Q_NPN_EBC, Q2 Q_PMOS_GSD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

Commit message: V0.2
Parts:
- added R13: 100k, Resistor_SMD:R_0603_1608Metric, symbol Device:R
- added R14, R15: 5.1k, Resistor_SMD:R_0603_1608Metric, symbol Device:R
- C15, C9: value 1000uf -> 470uf
- C6: value 1nf -> 1uf
- C7: value 2.2nf -> 2.2uf
- Q2: footprint Package_TO_SOT_SMD:SOT-23 -> KisonCommon:DFN-8-1EP_3x3mm_P0.65mm_EP1.7x2.05mm
- R10: value 470 -> 2.2k
Connections:
- wire segments 56 -> 60
Changed lines of the file:
@@
 P 9350 3250
 F 0 "C9" H 9468 3296 50  0000 L CNN
-F 1 "1000uf" H 9468 3205 50  0000 L CNN
+F 1 "470uf" H 9468 3205 50  0000 L CNN
 F 2 "Capacitor_THT:CP_Radial_D8.0mm_P3.50mm" H 9388 3100 50  0001 C CNN
 F 3 "~" H 9350 3250 50  0001 C CNN
@@
 P 8600 1350
 F 0 "C6" H 8715 1396 50  0000 L CNN
-F 1 "1nf" H 8715 1305 50  0000 L CNN
+F 1 "1uf" H 8715 1305 50  0000 L CNN
 F 2 "Capacitor_SMD:C_0603_1608Metric" H 8638 1200 50  0001 C CNN
 F 3 "~" H 8600 1350 50  0001 C CNN
@@
 P 9450 1350
 F 0 "C7" H 9565 1396 50  0000 L CNN
-F 1 "2.2nf" H 9565 1305 50  0000 L CNN
+F 1 "2.2uf" H 9565 1305 50  0000 L CNN
 F 2 "Capacitor_SMD:C_0603_1608Metric" H 9488 1200 50  0001 C CNN
 F 3 "~" H 9450 1350 50  0001 C CNN
@@
 	7800 2650 8050 2650
 $Comp
-L Connector:USB_C_Receptacle J9
-U 1 1 5F678410
-P 8150 4400
-F 0 "J9" H 8257 5667 50  0000 C CNN
-F 1 "USB_C_Receptacle" H 8257 5576 50  0000 C CNN
-F 2 "Connector_USB:USB_C_Receptacle_HRO_TYPE-C-31-M-12" H 8300 4400 50  0001 C CNN
-F 3 "https://www.usb.org/sites/default/files/documents/usb_type-c.zip" H 8300 4400 50  0001 C CNN
-	1    8150 4400
-	1    0    0    -1
-$EndComp
-$Comp
 L power:GND #PWR0110
 U 1 1 5F67D43F
@@
 Wire Wire Line
 	7850 6000 8150 6000
-Connection ~ 8150 6000
 $Comp
 L power:+5V #PWR0111
@@
 Wire Wire Line
 	1750 2000 2100 2000
-Text Label 1500 5950 2    50   ~ 0
+Text Label 1200 5950 2    50   ~ 0
 STEER_EN
 $Comp
 L Device:R R9
 U 1 1 5F598FE9
-P 1650 5950
-F 0 "R9" V 1443 5950 50  0000 C CNN
-F 1 "2.2k" V 1534 5950 50  0000 C CNN
-F 2 "Resistor_SMD:R_0603_1608Metric" V 1580 5950 50  0001 C CNN
-F 3 "~" H 1650 5950 50  0001 C CNN
-	1    1650 5950
+P 1350 5950
+F 0 "R9" V 1143 5950 50  0000 C CNN
+F 1 "2.2k" V 1234 5950 50  0000 C CNN
+F 2 "Resistor_SMD:R_0603_1608Metric" V 1280 5950 50  0001 C CNN
+F 3 "~" H 1350 5950 50  0001 C CNN
+	1    1350 5950
 	0    1    1    0
 $EndComp
@@
 	1    0    0    -1
 $EndComp
-$Comp
-L Device:R R10
-U 1 1 5F5A4164
-P 2100 5450
-F 0 "R10" H 2170 5496 50  0000 L CNN
-F 1 "470" H 2170 5405 50  0000 L CNN
-F 2 "Resistor_SMD:R_0603_1608Metric" V 2030 5450 50  0001 C CNN
-F 3 "~" H 2100 5450 50  0001 C CNN
-	1    2100 5450
-	1    0    0    -1
-$EndComp
 Wire Wire Line
 	2100 5600 2100 5750
-$Comp
-L Device:Q_PMOS_GSD Q2
-U 1 1 5F5A85F7
-P 2800 5750
-F 0 "Q2" H 3005 5704 50  0000 L CNN
-F 1 "Q_PMOS_GSD" H 3005 5795 50  0000 L CNN
-F 2 "Package_TO_SOT_SMD:SOT-23" H 3000 5850 50  0001 C CNN
-F 3 "~" H 2800 5750 50  0001 C CNN
-	1    2800 5750
-	1    0    0    1
-$EndComp
 Wire Wire Line
 	2100 5750 2600 5750
@@
 Wire Wire Line
 	2100 5300 2900 5300
-Wire Wire Line
-	2900 5300 2900 5550
 Connection ~ 2100 5300
 Text Label 4200 2000 2    50   ~ 0
@@
 Text Label 9350 3100 2    50   ~ 0
 VOutput
-Text Label 2900 5950 2    50   ~ 0
+Text Label 2900 5950 3    50   ~ 0
 VOutput
 $Comp
@@
 P 9350 4000
 F 0 "C15" H 9468 4046 50  0000 L CNN
-F 1 "1000uf" H 9468 3955 50  0000 L CNN
+F 1 "470uf" H 9468 3955 50  0000 L CNN
 F 2 "Capacitor_THT:CP_Radial_D8.0mm_P3.50mm" H 9388 3850 50  0001 C CNN
 F 3 "~" H 9350 4000 50  0001 C CNN
@@
 	-1   0    0    1
 $EndComp
+$Comp
+L Device:R R13
+U 1 1 5F590065
+P 1500 6100
+F 0 "R13" H 1570 6146 50  0000 L CNN
+F 1 "100k" H 1570 6055 50  0000 L CNN
+F 2 "Resistor_SMD:R_0603_1608Metric" V 1430 6100 50  0001 C CNN
+F 3 "~" H 1500 6100 50  0001 C CNN
+	1    1500 6100
+	1    0    0    -1
+$EndComp
+Wire Wire Line
+	1500 5950 1800 5950
+Connection ~ 1500 5950
+$Comp
+L power:GND #PWR0113
+U 1 1 5F59A3B1
+P 1500 6250
+F 0 "#PWR0113" H 1500 6000 50  0001 C CNN
+F 1 "GND" V 1505 6122 50  0000 R CNN
+F 2 "" H 1500 6250 50  0001 C CNN
+F 3 "" H 1500 6250 50  0001 C CNN
+	1    1500 6250
+	1    0    0    -1
+$EndComp
+Wire Wire Line
+	2900 5300 2900 5550
+$Comp
+L Device:Q_PMOS_GSD Q2
+U 1 1 5F5A85F7
+P 2800 5750
+F 0 "Q2" H 3005 5704 50  0000 L CNN
+F 1 "Q_PMOS_GSD" H 3005 5795 50  0000 L CNN
+F 2 "KisonCommon:DFN-8-1EP_3x3mm_P0.65mm_EP1.7x2.05mm" H 3000 5850 50  0001 C CNN
+F 3 "~" H 2800 5750 50  0001 C CNN
+	1    2800 5750
+	1    0    0    1
+$EndComp
+Connection ~ 8150 6000
+$Comp
+L Connector:USB_C_Receptacle J9
+U 1 1 5F678410
+P 8150 4400
+F 0 "J9" H 8257 5667 50  0000 C CNN
+F 1 "USB_C_Receptacle" H 8257 5576 50  0000 C CNN
+F 2 "Connector_USB:USB_C_Receptacle_HRO_TYPE-C-31-M-12" H 8300 4400 50  0001 C CNN
+F 3 "https://www.usb.org/sites/default/files/documents/usb_type-c.zip" H 8300 4400 50  0001 C CNN
+	1    8150 4400
+	1    0    0    -1
+$EndComp
+Wire Wire Line
+	8750 3900 8750 4000
+Wire Wire Line
+	8750 4100 8750 4200
+$Comp
+L Device:R R14
+U 1 1 5F59C17E
+P 8900 3600
+F 0 "R14" V 8693 3600 50  0000 C CNN
+F 1 "5.1k" V 8784 3600 50  0000 C CNN
+F 2 "Resistor_SMD:R_0603_1608Metric" V 8830 3600 50  0001 C CNN
+F 3 "~" H 8900 3600 50  0001 C CNN
+	1    8900 3600
+	0    1    1    0
+$EndComp
+$Comp
+L Device:R R15
+U 1 1 5F59C4FC
+P 8900 3700
+F 0 "R15" V 9000 3700 50  0000 C CNN
+F 1 "5.1k" V 9100 3700 50  0000 C CNN
+F 2 "Resistor_SMD:R_0603_1608Metric" V 8830 3700 50  0001 C CNN
+F 3 "~" H 8900 3700 50  0001 C CNN
+	1    8900 3700
+	0    1    1    0
+$EndComp
+Wire Wire Line
+	9050 3600 9050 3700
+$Comp
+L power:GND #PWR025
+U 1 1 5F5A897B
+P 9050 3600
+F 0 "#PWR025" H 9050 3350 50  0001 C CNN
+F 1 "GND" V 9055 3472 50  0000 R CNN
+F 2 "" H 9050 3600 50  0001 C CNN
+F 3 "" H 9050 3600 50  0001 C CNN
+	1    9050 3600
+	0    -1   -1   0
+$EndComp
+Connection ~ 9050 3600
+$Comp
+L Device:R R10
+U 1 1 5F5A4164
+P 2100 5450
+F 0 "R10" H 2170 5496 50  0000 L CNN
+F 1 "2.2k" H 2170 5405 50  0000 L CNN
+F 2 "Resistor_SMD:R_0603_1608Metric" V 2030 5450 50  0001 C CNN
+F 3 "~" H 2100 5450 50  0001 C CNN
+	1    2100 5450
+	1    0    0    -1
+$EndComp
 $EndSCHEMATC

Commit message: V0.29
Parts:
- L1: footprint Inductor_SMD:L_1008_2520Metric -> Inductor_SMD:L_6.3x6.3_H3
Changed lines of the file:
@@
 F 0 "L1" V 8269 2750 50  0000 C CNN
 F 1 "4.7uh" V 8360 2750 50  0000 C CNN
-F 2 "Inductor_SMD:L_1008_2520Metric" H 8450 2750 50  0001 C CNN
+F 2 "Inductor_SMD:L_6.3x6.3_H3" H 8450 2750 50  0001 C CNN
 F 3 "~" H 8450 2750 50  0001 C CNN
 	1    8450 2750

Commit message: V1.0
Parts:
- removed Q3: Q_NPN_EBC, Package_TO_SOT_SMD:SOT-23, symbol Device:Q_NPN_EBC
- added Q3: Q_PMOS_GSD, KisonCommon:DFN-8-1EP_3x3mm_P0.65mm_EP1.7x2.05mm, symbol Device:Q_PMOS_GSD
- J2: footprint Connector_PinHeader_1.27mm:PinHeader_1x05_P1.27mm_Vertical -> Connector_PinHeader_2.54mm:PinHeader_1x05_P2.54mm_Vertical
Changed lines of the file:
@@
 F 0 "J2" H 2980 892 50  0000 L CNN
 F 1 "Conn_01x05" H 2980 801 50  0000 L CNN
-F 2 "Connector_PinHeader_1.27mm:PinHeader_1x05_P1.27mm_Vertical" H 2900 850 50  0001 C CNN
+F 2 "Connector_PinHeader_2.54mm:PinHeader_1x05_P2.54mm_Vertical" H 2900 850 50  0001 C CNN
 F 3 "~" H 2900 850 50  0001 C CNN
 	1    2900 850
@@
 LEDA_32
 $Comp
-L Device:Q_NPN_EBC Q3
-U 1 1 5F5C89CF
-P 4900 6350
-F 0 "Q3" H 5091 6396 50  0000 L CNN
-F 1 "Q_NPN_EBC" H 5091 6305 50  0000 L CNN
-F 2 "Package_TO_SOT_SMD:SOT-23" H 5100 6450 50  0001 C CNN
-F 3 "~" H 4900 6350 50  0001 C CNN
-	1    4900 6350
-	1    0    0    -1
-$EndComp
-$Comp
 L power:+3V3 #PWR010
 U 1 1 5F5C9609
@@
 	0    1    1    0
 $EndComp
-Wire Wire Line
-	4250 6350 4500 6350
-$Comp
-L Device:R R12
-U 1 1 5F60365C
-P 4500 6500
-F 0 "R12" H 4570 6546 50  0000 L CNN
-F 1 "10k" H 4570 6455 50  0000 L CNN
-F 2 "Resistor_SMD:R_0603_1608Metric" V 4430 6500 50  0001 C CNN
-F 3 "~" H 4500 6500 50  0001 C CNN
-	1    4500 6500
-	1    0    0    -1
-$EndComp
-Connection ~ 4500 6350
-Wire Wire Line
-	4500 6350 4700 6350
+$Comp
+L Device:R R13
+U 1 1 5F590065
+P 1500 6100
+F 0 "R13" H 1570 6146 50  0000 L CNN
+F 1 "100k" H 1570 6055 50  0000 L CNN
+F 2 "Resistor_SMD:R_0603_1608Metric" V 1430 6100 50  0001 C CNN
+F 3 "~" H 1500 6100 50  0001 C CNN
+	1    1500 6100
+	1    0    0    -1
+$EndComp
+Wire Wire Line
+	1500 5950 1800 5950
+Connection ~ 1500 5950
+$Comp
+L power:GND #PWR0113
+U 1 1 5F59A3B1
+P 1500 6250
+F 0 "#PWR0113" H 1500 6000 50  0001 C CNN
+F 1 "GND" V 1505 6122 50  0000 R CNN
+F 2 "" H 1500 6250 50  0001 C CNN
+F 3 "" H 1500 6250 50  0001 C CNN
+	1    1500 6250
+	1    0    0    -1
+$EndComp
+Wire Wire Line
+	2900 5300 2900 5550
+$Comp
+L Device:Q_PMOS_GSD Q2
+U 1 1 5F5A85F7
+P 2800 5750
+F 0 "Q2" H 3005 5704 50  0000 L CNN
+F 1 "Q_PMOS_GSD" H 3005 5795 50  0000 L CNN
+F 2 "KisonCommon:DFN-8-1EP_3x3mm_P0.65mm_EP1.7x2.05mm" H 3000 5850 50  0001 C CNN
+F 3 "~" H 2800 5750 50  0001 C CNN
+	1    2800 5750
+	1    0    0    1
+$EndComp
+Connection ~ 8150 6000
+$Comp
+L Connector:USB_C_Receptacle J9
+U 1 1 5F678410
+P 8150 4400
+F 0 "J9" H 8257 5667 50  0000 C CNN
+F 1 "USB_C_Receptacle" H 8257 5576 50  0000 C CNN
+F 2 "Connector_USB:USB_C_Receptacle_HRO_TYPE-C-31-M-12" H 8300 4400 50  0001 C CNN
+F 3 "https://www.usb.org/sites/default/files/documents/usb_type-c.zip" H 8300 4400 50  0001 C CNN
+	1    8150 4400
+	1    0    0    -1
+$EndComp
+Wire Wire Line
+	8750 3900 8750 4000
+Wire Wire Line
+	8750 4100 8750 4200
+$Comp
+L Device:R R14
+U 1 1 5F59C17E
+P 8900 3600
+F 0 "R14" V 8693 3600 50  0000 C CNN
+F 1 "5.1k" V 8784 3600 50  0000 C CNN
+F 2 "Resistor_SMD:R_0603_1608Metric" V 8830 3600 50  0001 C CNN
+F 3 "~" H 8900 3600 50  0001 C CNN
+	1    8900 3600
+	0    1    1    0
+$EndComp
+$Comp
+L Device:R R15
+U 1 1 5F59C4FC
+P 8900 3700
+F 0 "R15" V 9000 3700 50  0000 C CNN
+F 1 "5.1k" V 9100 3700 50  0000 C CNN
+F 2 "Resistor_SMD:R_0603_1608Metric" V 8830 3700 50  0001 C CNN
+F 3 "~" H 8900 3700 50  0001 C CNN
+	1    8900 3700
+	0    1    1    0
+$EndComp
+Wire Wire Line
+	9050 3600 9050 3700
+$Comp
+L power:GND #PWR025
+U 1 1 5F5A897B
+P 9050 3600
+F 0 "#PWR025" H 9050 3350 50  0001 C CNN
+F 1 "GND" V 9055 3472 50  0000 R CNN
+F 2 "" H 9050 3600 50  0001 C CNN
+F 3 "" H 9050 3600 50  0001 C CNN
+	1    9050 3600
+	0    -1   -1   0
+$EndComp
+Connection ~ 9050 3600
+$Comp
+L Device:R R10
+U 1 1 5F5A4164
+P 2100 5450
+F 0 "R10" H 2170 5496 50  0000 L CNN
+F 1 "2.2k" H 2170 5405 50  0000 L CNN
+F 2 "Resistor_SMD:R_0603_1608Metric" V 2030 5450 50  0001 C CNN
+F 3 "~" H 2100 5450 50  0001 C CNN
+	1    2100 5450
+	1    0    0    -1
+$EndComp
 $Comp
 L power:+3V3 #PWR0109
@@
 	-1   0    0    1
 $EndComp
-$Comp
-L Device:R R13
-U 1 1 5F590065
-P 1500 6100
-F 0 "R13" H 1570 6146 50  0000 L CNN
-F 1 "100k" H 1570 6055 50  0000 L CNN
-F 2 "Resistor_SMD:R_0603_1608Metric" V 1430 6100 50  0001 C CNN
-F 3 "~" H 1500 6100 50  0001 C CNN
-	1    1500 6100
-	1    0    0    -1
-$EndComp
-Wire Wire Line
-	1500 5950 1800 5950
-Connection ~ 1500 5950
-$Comp
-L power:GND #PWR0113
-U 1 1 5F59A3B1
-P 1500 6250
-F 0 "#PWR0113" H 1500 6000 50  0001 C CNN
-F 1 "GND" V 1505 6122 50  0000 R CNN
-F 2 "" H 1500 6250 50  0001 C CNN
-F 3 "" H 1500 6250 50  0001 C CNN
-	1    1500 6250
-	1    0    0    -1
-$EndComp
-Wire Wire Line
-	2900 5300 2900 5550
-$Comp
-L Device:Q_PMOS_GSD Q2
-U 1 1 5F5A85F7
-P 2800 5750
-F 0 "Q2" H 3005 5704 50  0000 L CNN
-F 1 "Q_PMOS_GSD" H 3005 5795 50  0000 L CNN
-F 2 "KisonCommon:DFN-8-1EP_3x3mm_P0.65mm_EP1.7x2.05mm" H 3000 5850 50  0001 C CNN
-F 3 "~" H 2800 5750 50  0001 C CNN
-	1    2800 5750
+Wire Wire Line
+	4500 6350 4700 6350
+Wire Wire Line
+	4250 6350 4500 6350
+Connection ~ 4500 6350
+$Comp
+L Device:R R12
+U 1 1 5F60365C
+P 4500 6500
+F 0 "R12" H 4570 6546 50  0000 L CNN
+F 1 "10k" H 4570 6455 50  0000 L CNN
+F 2 "Resistor_SMD:R_0603_1608Metric" V 4430 6500 50  0001 C CNN
+F 3 "~" H 4500 6500 50  0001 C CNN
+	1    4500 6500
+	1    0    0    -1
+$EndComp
+$Comp
+L Device:Q_PMOS_GSD Q3
+U 1 1 5F593D85
+P 4900 6350
+F 0 "Q3" H 5105 6304 50  0000 L CNN
+F 1 "Q_PMOS_GSD" H 5105 6395 50  0000 L CNN
+F 2 "KisonCommon:DFN-8-1EP_3x3mm_P0.65mm_EP1.7x2.05mm" H 5100 6450 50  0001 C CNN
+F 3 "~" H 4900 6350 50  0001 C CNN
+	1    4900 6350
 	1    0    0    1
 $EndComp
-Connection ~ 8150 6000
-$Comp
-L Connector:USB_C_Receptacle J9
-U 1 1 5F678410
-P 8150 4400
-F 0 "J9" H 8257 5667 50  0000 C CNN
-F 1 "USB_C_Receptacle" H 8257 5576 50  0000 C CNN
-F 2 "Connector_USB:USB_C_Receptacle_HRO_TYPE-C-31-M-12" H 8300 4400 50  0001 C CNN
-F 3 "https://www.usb.org/sites/default/files/documents/usb_type-c.zip" H 8300 4400 50  0001 C CNN
-	1    8150 4400
-	1    0    0    -1
-$EndComp
-Wire Wire Line
-	8750 3900 8750 4000
-Wire Wire Line
-	8750 4100 8750 4200
-$Comp
-L Device:R R14
-U 1 1 5F59C17E
-P 8900 3600
-F 0 "R14" V 8693 3600 50  0000 C CNN
-F 1 "5.1k" V 8784 3600 50  0000 C CNN
-F 2 "Resistor_SMD:R_0603_1608Metric" V 8830 3600 50  0001 C CNN
-F 3 "~" H 8900 3600 50  0001 C CNN
-	1    8900 3600
-	0    1    1    0
-$EndComp
-$Comp
-L Device:R R15
-U 1 1 5F59C4FC
-P 8900 3700
-F 0 "R15" V 9000 3700 50  0000 C CNN
-F 1 "5.1k" V 9100 3700 50  0000 C CNN
-F 2 "Resistor_SMD:R_0603_1608Metric" V 8830 3700 50  0001 C CNN
-F 3 "~" H 8900 3700 50  0001 C CNN
-	1    8900 3700
-	0    1    1    0
-$EndComp
-Wire Wire Line
-	9050 3600 9050 3700
-$Comp
-L power:GND #PWR025
-U 1 1 5F5A897B
-P 9050 3600
-F 0 "#PWR025" H 9050 3350 50  0001 C CNN
-F 1 "GND" V 9055 3472 50  0000 R CNN
-F 2 "" H 9050 3600 50  0001 C CNN
-F 3 "" H 9050 3600 50  0001 C CNN
-	1    9050 3600
-	0    -1   -1   0
-$EndComp
-Connection ~ 9050 3600
-$Comp
-L Device:R R10
-U 1 1 5F5A4164
-P 2100 5450
-F 0 "R10" H 2170 5496 50  0000 L CNN
-F 1 "2.2k" H 2170 5405 50  0000 L CNN
-F 2 "Resistor_SMD:R_0603_1608Metric" V 2030 5450 50  0001 C CNN
-F 3 "~" H 2100 5450 50  0001 C CNN
-	1    2100 5450
-	1    0    0    -1
-$EndComp
 $EndSCHEMATC

Commit message: V1.1
Changed lines of the file:
@@
 Text Label 1400 950  0    50   ~ 0
 STM_SWDIO
+Text Label 3400 4300 0    50   ~ 0
+STM_SWCLK
 Text Label 3400 4200 0    50   ~ 0
-STM_SWCLK
-Text Label 3400 4300 0    50   ~ 0
 STM_SWDIO
 Connection ~ 2900 4600

Commit message: V1.2
Parts:
- removed Q1: Q_NPN_EBC, Package_TO_SOT_SMD:SOT-23, symbol Device:Q_NPN_EBC
- added H13: 1mm Hole, KisonCommon:1mm Hole, symbol Mechanical:MountingHole
- added H5, H6, H7: MountingHole, MountingHole:MountingHole_2.2mm_M2_DIN965, symbol Mechanical:MountingHole
- added J10: Conn_02x03_Odd_Even, Connector_PinHeader_1.27mm:PinHeader_2x03_P1.27mm_Vertical, symbol Connector_Generic:Conn_02x03_Odd_Even
- added Q1: Q_NPN_BEC, Package_TO_SOT_SMD:SOT-23, symbol Device:Q_NPN_BEC
- added R16, R17, R19: 10k, Resistor_SMD:R_0603_1608Metric, symbol Device:R
- added R18: 5.1k, Resistor_SMD:R_0603_1608Metric, symbol Device:R
- added U4: LM321, Package_TO_SOT_SMD:SOT-23-5, symbol Amplifier_Operational:LM321
- H1, H2, H3, H4: footprint MountingHole:MountingHole_3mm -> MountingHole:MountingHole_2.2mm_M2_DIN965
Connections:
- wire segments 60 -> 69

Commit message: Update UART IRQ
Changed lines of the file:
@@
 Text Label 3400 3900 0    50   ~ 0
 UART_32RX
+Text Label 4750 4600 2    50   ~ 0
+UART_32TX
 Text Label 4750 4700 2    50   ~ 0
-UART_32TX
-Text Label 4750 4600 2    50   ~ 0
 UART_32RX
 Text Label 4750 3600 2    50   ~ 0

Commit message: Embeded Ver 1.0
Parts:
- added R20, R21: 0, Capacitor_SMD:C_0603_1608Metric, symbol Device:R
Connections:
- net labels added: STEER_EN_8266, STEER_PWM_8266
- wire segments 69 -> 73
Changed lines of the file:
@@
 	0    1    1    0
 $EndComp
-Text Label 4200 2000 2    50   ~ 0
+Text Label 4050 2000 2    50   ~ 0
 STEER_PWM
 $Comp
@@
 Wire Wire Line
 	1750 2000 2100 2000
-Text Label 1000 5600 2    50   ~ 0
+Text Label 900  5600 2    50   ~ 0
 STEER_EN
 $Comp
@@
 	1    0    0    -1
 $EndComp
-Wire Wire Line
-	1300 5600 1600 5600
 Connection ~ 1300 5600
 $Comp
@@
 	-1   0    0    1
 $EndComp
+$Comp
+L Device:R R20
+U 1 1 5F7ADBF5
+P 950 5450
+F 0 "R20" H 1020 5496 50  0000 L CNN
+F 1 "0" H 1020 5405 50  0000 L CNN
+F 2 "Capacitor_SMD:C_0603_1608Metric" V 880 5450 50  0001 C CNN
+F 3 "~" H 950 5450 50  0001 C CNN
+	1    950  5450
+	1    0    0    -1
+$EndComp
+Wire Wire Line
+	900  5600 950  5600
+Wire Wire Line
+	1300 5600 1600 5600
+Wire Wire Line
+	950  5600 1000 5600
+Connection ~ 950  5600
+Text Label 950  5300 0    50   ~ 0
+STEER_EN_8266
+Text Label 4750 4500 2    50   ~ 0
+STEER_EN_8266
+$Comp
+L Device:R R21
+U 1 1 5F7C7CE7
+P 4100 1850
+F 0 "R21" H 4170 1896 50  0000 L CNN
+F 1 "0" H 4170 1805 50  0000 L CNN
+F 2 "Capacitor_SMD:C_0603_1608Metric" V 4030 1850 50  0001 C CNN
+F 3 "~" H 4100 1850 50  0001 C CNN
+	1    4100 1850
+	1    0    0    -1
+$EndComp
+Wire Wire Line
+	4050 2000 4100 2000
+Connection ~ 4100 2000
+Wire Wire Line
+	4100 2000 4200 2000
+Text Label 4100 1700 0    50   ~ 0
+STEER_PWM_8266
+Text Label 4750 4400 2    50   ~ 0
+STEER_PWM_8266
 $EndSCHEMATC

Commit message: PCBV3.0
Parts:
- removed C15, C9: 470uf, Capacitor_THT:CP_Radial_D8.0mm_P3.50mm, symbol Device:CP
- removed C16: 1000uf, Capacitor_THT:CP_Radial_D8.0mm_P3.50mm, symbol Device:CP
- removed J10: Conn_02x03_Odd_Even, Connector_PinHeader_1.27mm:PinHeader_2x03_P1.27mm_Vertical, symbol Connector_Generic:Conn_02x03_Odd_Even
- added D1: LED_RGB, LED_SMD:LED_RGB_5050-6, symbol Device:LED_RGB
- added D2, D3, D4: LED, LED_SMD:LED_0603_1608Metric, symbol Device:LED
- added H8: 0.7mm Hole, KisonCommon:0.7mmInR Hole, symbol Mechanical:MountingHole
- added R22, R23, R24, R27, R28, R29: 2.2k, Resistor_SMD:R_0603_1608Metric, symbol Device:R
- added R25, R26: 0, Resistor_SMD:R_0603_1608Metric, symbol Device:R
- H13: value 1mm Hole -> 0.7mm Hole; footprint KisonCommon:1mm Hole -> KisonCommon:0.7mmInR Hole
- R20, R21: footprint Capacitor_SMD:C_0603_1608Metric -> Resistor_SMD:R_0603_1608Metric
Connections:
- net labels added: RGB_B, RGB_G, RGB_R
- wire segments 73 -> 91
